File: fkb-109j-big/fkb-109j-big.kicad_sch (KiCad schematic)
At the start: 273 parts, among them J1 Conn_02x07_Counter_Clockwise, J2 Conn_02x07_Counter_Clockwise, J3 Conn_01x01_Pin, J4 Conn_01x01_Pin, J5 Conn_01x05_Pin

Commit message: layout... done?
Parts:
- removed J5: Conn_01x05_Pin, Connector_PinHeader_2.00mm:PinHeader_1x05_P2.00mm_Vertical, symbol Connector:Conn_01x05_Pin
- removed R14, R15, R16, R23, R24, R25, R26: R, Resistor_THT:R_Axial_DIN0207_L6.3mm_D2.5mm_P10.16mm_Horizontal, symbol Device:R
- added J10: Conn_01x04, Connector_PinHeader_2.00mm:PinHeader_1x04_P2.00mm_Vertical, symbol Connector_Generic:Conn_01x04
- added J5, J6, J7: Conn_01x05, Connector_PinHeader_2.00mm:PinHeader_1x05_P2.00mm_Vertical, symbol Connector_Generic:Conn_01x05
- added J8, J9: Conn_01x03, Connector_PinHeader_2.00mm:PinHeader_1x03_P2.00mm_Vertical, symbol Connector_Generic:Conn_01x03
Connections:
- net COL14_BOTTOM: now also J9.1 (Pin_1)
- net COL15_BOTTOM: now also J9.2 (Pin_2)
- net COL16_BOTTOM: now also J9.3 (Pin_3)
- net COL17_BOTTOM: now also J10.1 (Pin_1)
- net COL18_BOTTOM: now also J10.2 (Pin_2)
- net COL19_BOTTOM: now also J10.3 (Pin_3)
- net COL20_BOTTOM: now also J10.4 (Pin_4)
- net ROW4_RIGHT: now reaches D102.1 (K), D106.1 (K), D111.1 (K), D97.1 (K)
- net ROW4_RIGHT: now also J7.4 (Pin_4)
- net COL15_TOP: now reaches MX_SCRLK1.1 (COL), MX_SCRLK2.2 (ROW)
- net COL15_TOP: now also J8.2 (Pin_2)
- net ROW1_MID: now reaches D82.1 (K), D86.1 (K), D91.1 (K)
- net ROW1_MID: now also J6.1 (Pin_1)
- net ROW1_RIGHT: now reaches D103.1 (K), D108.1 (K), D94.1 (K), D99.1 (K)
- net ROW1_RIGHT: now also J7.1 (Pin_1)
- net ROW5_MID: now reaches D84.1 (K), D89.1 (K), D93.1 (K)
- net ROW5_MID: now also J6.5 (Pin_5)
- net ROW2_MID: now reaches D83.1 (K), D87.1 (K), D92.1 (K)
- net ROW2_MID: now also J6.2 (Pin_2)
- net COL14_TOP: now reaches MX_PSCRN1.1 (COL), MX_PSCRN2.2 (ROW)
- net COL14_TOP: now also J8.1 (Pin_1)
- net ROW5_RIGHT: now reaches D107.1 (K), D98.1 (K)
- net ROW5_RIGHT: now also J7.5 (Pin_5)
- net ROW2_RIGHT: now reaches D100.1 (K), D104.1 (K), D109.1 (K), D95.1 (K)
- net ROW2_RIGHT: now also J7.2 (Pin_2)
- net ROW3_RIGHT: now reaches D101.1 (K), D105.1 (K), D110.1 (K), D96.1 (K)
- net ROW3_RIGHT: now also J7.3 (Pin_3)
- net COL16_TOP: now reaches MX_PSBRK1.1 (COL), MX_PSBRK2.2 (ROW)
- net COL16_TOP: now also J8.3 (Pin_3)
- net ROW4_MID: now reaches D88.1 (K)
- net ROW4_MID: now also J6.4 (Pin_4)
- net ROW1 renamed ROW1_LEFT
- net ROW1_LEFT: now also J5.1 (Pin_1)
- net ROW2 renamed ROW2_LEFT
- net ROW2_LEFT: now also J5.2 (Pin_2)
- net ROW3 renamed ROW3_LEFT
- net ROW3_LEFT: now also J5.3 (Pin_3)
- net ROW4 renamed ROW4_LEFT
- net ROW4_LEFT: now also J5.4 (Pin_4)
- net ROW5 renamed ROW5_LEFT
- net ROW5_LEFT: now also J5.5 (Pin_5)
- new net ROW3_MID: J6.3 (Pin_3)
Other:
- moved on the sheet: J1, J2
