File: fkb-109j-big/fkb-109j-big.kicad_pcb (KiCad board)
At the start: 2 copper layers, 429.1 x 119.3 mm, 282 parts, among them J1 Conn_02x07_Counter_Clockwise, J2 Conn_02x07_Counter_Clockwise, J3 Conn_01x01_Pin, J4 Conn_01x01_Pin, J5 Conn_01x05_Pin

Commit message: layout... done?
Parts:
- removed R14, R15, R16, R23, R24, R25, R26: R, Resistor_THT:R_Axial_DIN0207_L6.3mm_D2.5mm_P10.16mm_Horizontal
- added J10: Conn_01x04, Connector_PinHeader_2.00mm:PinHeader_1x04_P2.00mm_Vertical, F.Cu at (499.2, 53.7)
- added J6: Conn_01x05, Connector_PinHeader_2.00mm:PinHeader_1x05_P2.00mm_Vertical, F.Cu at (422.2, 55.9)
- added J7: Conn_01x05, Connector_PinHeader_2.00mm:PinHeader_1x05_P2.00mm_Vertical, F.Cu at (484.4, 53.7)
- added J8: Conn_01x03, Connector_PinHeader_2.00mm:PinHeader_1x03_P2.00mm_Vertical, F.Cu at (447.1, 29.6)
- added J9: Conn_01x03, Connector_PinHeader_2.00mm:PinHeader_1x03_P2.00mm_Vertical, F.Cu at (457.1, 53.7)
- J5: value Conn_01x05_Pin -> Conn_01x05
Connections:
- net Net-(D100-K) renamed ROW2_RIGHT
- net Net-(D101-K) renamed ROW3_RIGHT
- net Net-(D102-K) renamed ROW4_RIGHT
- net Net-(D103-K) renamed ROW1_RIGHT
- net Net-(D107-K) renamed ROW5_RIGHT
- net Net-(D82-K) renamed ROW1_MID
- net Net-(D83-K) renamed ROW2_MID
- net Net-(D84-K) renamed ROW5_MID
- net Net-(MX_PSBRK1-COL) renamed COL16_TOP
- net Net-(MX_PSCRN1-COL) renamed COL14_TOP
- net Net-(MX_SCRLK1-COL) renamed COL15_TOP
- net ROW1 renamed ROW1_LEFT
- net ROW2 renamed ROW2_LEFT
- net ROW3 renamed ROW3_LEFT
- net ROW4 renamed ROW4_LEFT
- net ROW5 renamed ROW5_LEFT
- D88 pad 1: Net-(D88-K) -> ROW4_MID
Routing:
- net COL13_BOTTOM: track 258.5 -> 541.9 mm
- net Net-(D79-A): track 11.3 -> 280.0 mm
- net ROW5_RIGHT: track 20.6 -> 122.4 mm
- net ROW5_MID: track 36.8 -> 126.8 mm
- net ROW4_MID: track 0.00 -> 81.0 mm
- net ROW4_RIGHT: track 64.2 -> 139.5 mm
- net ROW3_RIGHT: track 55.6 -> 113.7 mm
- net COL20_BOTTOM: track 84.6 -> 128.3 mm
- net ROW2_RIGHT: track 55.7 -> 96.7 mm
- net ROW2_MID: track 29.2 -> 68.2 mm
- net COL14_BOTTOM: track 76.2 -> 107.0 mm
- net COL19_BOTTOM: track 76.2 -> 102.9 mm
- net ROW1_RIGHT: track 55.5 -> 81.6 mm
- net ROW1_MID: track 28.6 -> 52.4 mm
- net COL14_TOP: track 2.62 -> 23.6 mm
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
Commit message: add some holes.
Routing:
- net COL14_BOTTOM: track 107.0 -> 109.8 mm
- net ROW5_MID: track 126.8 -> 127.8 mm
Other:
- outline, holes or cut-outs redrawn
Changed lines of the file:
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@@
     )
   )
+  (gr_circle (center 377.825 138.1125) (end 383.325 138.1125)
+    (stroke (width 0.1) (type default)) (fill none) (layer "B.SilkS"))
   (gr_line (start 415.925 32.825) (end 415.925 28.3375)
     (stroke (width 0.1) (type default)) (layer "Edge.Cuts"))
-  (gr_line (start 144.2 47.4) (end 130.175 47.3875)
-    (stroke (width 0.1) (type default)) (layer "Edge.Cuts"))
-  (gr_line (start 130.175 28.3375) (end 130.175 47.3875)
+  (gr_line (start 130.175 28.3375) (end 130.175 46.1375)
+    (stroke (width 0.1) (type default)) (layer "Edge.Cuts"))
+  (gr_line (start 131.449748 47.387255) (end 144.2 47.4)
     (stroke (width 0.1) (type default)) (layer "Edge.Cuts"))
   (gr_line (start 478.1 133.6) (end 478.075 147.6375)
@@
   (gr_arc (start 478.1 133.6) (mid 480.587438 131.087563) (end 483.099875 133.575001)
     (stroke (width 0.1) (type default)) (layer "Edge.Cuts"))
+  (gr_circle (center 449.5 103.5625) (end 451.5 103.5625)
+    (stroke (width 0.1) (type default)) (fill none) (layer "Edge.Cuts"))
   (gr_line (start 401.9 52.4) (end 415.925 52.3875)
     (stroke (width 0.1) (type default)) (layer "Edge.Cuts"))
@@
   (gr_line (start 420.925 147.6375) (end 478.075 147.6375)
     (stroke (width 0.1) (type default)) (layer "Edge.Cuts"))
+  (gr_arc (start 131.449748 47.387255) (mid 130.553541 47.026387) (end 130.175 46.1375)
+    (stroke (width 0.1) (type default)) (layer "Edge.Cuts"))
   (gr_line (start 415.925 28.3375) (end 130.175 28.3375)
     (stroke (width 0.1) (type default)) (layer "Edge.Cuts"))
   (gr_line (start 420.925 123.6) (end 420.925 76.45)
     (stroke (width 0.1) (type default)) (layer "Edge.Cuts"))
+  (gr_circle (center 474.4 112.612) (end 476.4 112.612)
+    (stroke (width 0.1) (type default)) (fill none) (layer "Edge.Cuts"))
   (gr_line (start 444.5 52.375) (end 420.925 52.3875)
     (stroke (width 0.1) (type default)) (layer "Edge.Cuts"))
@@
   (gr_line (start 420.925 28.3375) (end 420.925 32.825)
     (stroke (width 0.1) (type default)) (layer "Edge.Cuts"))
+  (gr_circle (center 430.45 117.9) (end 435.95 117.9)
+    (stroke (width 0.1) (type default)) (fill none) (layer "Edge.Cuts"))
   (gr_line (start 483.075 147.6375) (end 559.275 147.6375)
     (stroke (width 0.1) (type default)) (layer "Edge.Cuts"))
@@
   (segment (start 164.0625 116.5125) (end 166.0125 114.5625) (width 0.25) (layer "B.Cu") (net 127))
   (segment (start 156.05 89.7) (end 156.05 112.15061) (width 0.25) (layer "B.Cu") (net 127))
-  (segment (start 427.95 57.9125) (end 427.95 134.1125) (width 0.25) (layer "F.Cu") (net 128))
+  (segment (start 427.95 76.9625) (end 424.622478 80.290022) (width 0.25) (layer "F.Cu") (net 128))
+  (segment (start 424.622478 80.290022) (end 424.622478 130.784978) (width 0.25) (layer "F.Cu") (net 128))
+  (segment (start 424.622478 130.784978) (end 427.95 134.1125) (width 0.25) (layer "F.Cu") (net 128))
+  (segment (start 427.95 57.9125) (end 427.95 76.9625) (width 0.25) (layer "F.Cu") (net 128))
   (segment (start 430.39939 57.9125) (end 427.95 57.9125) (width 0.25) (layer "B.Cu") (net 128))
   (segment (start 434.61189 53.7) (end 430.39939 57.9125) (width 0.25) (layer "B.Cu") (net 128))
@@
   (segment (start 439.975 146.52625) (end 476.63375 146.52625) (width 0.25) (layer "F.Cu") (net 156))
   (segment (start 476.63375 146.52625) (end 476.75 146.41) (width 0.25) (layer "F.Cu") (net 156))
-  (segment (start 422.25 63.9) (end 422.25 119.590259) (width 0.25) (layer "B.Cu") (net 156))
-  (segment (start 429.4 135.95125) (end 439.975 146.52625) (width 0.25) (layer "B.Cu") (net 156))
-  (segment (start 422.25 119.590259) (end 429.4 126.740259) (width 0.25) (layer "B.Cu") (net 156))
-  (segment (start 429.4 126.740259) (end 429.4 135.95125) (width 0.25) (layer "B.Cu") (net 156))
+  (segment (start 438.27625 146.52625) (end 439.975 146.52625) (width 0.25) (layer "B.Cu") (net 156))
+  (segment (start 422.25 63.9) (end 422.25 130.5) (width 0.25) (layer "B.Cu") (net 156))
+  (segment (start 422.25 130.5) (end 438.27625 146.52625) (width 0.25) (layer "B.Cu") (net 156))
   (segment (start 422.25 61.9) (end 423.25 62.9) (width 0.25) (layer "B.Cu") (net 157))
   (segment (start 459.025 125.03689) (end 459.025 127.635) (width 0.25) (layer "B.Cu") (net 157))

Commit message: add umu; minor cleanup.
Parts:
- added G***: LOGO, umu:umu, B.Cu at (456.7, 126.0)
- moved J8 9.90 mm to (457.1, 29.6)
- moved J6 1.85 mm to (422.2, 54.0)
- moved J7 0.35 mm to (484.4, 54.0)
Routing:
- net COL14_TOP: track 23.6 -> 33.5 mm
- net COL16_TOP: track 19.3 -> 9.39 mm
- net COL15_TOP: track 7.77 -> 16.4 mm
- net ROW5_MID: track 127.8 -> 129.6 mm
- net ROW4_MID: track 81.0 -> 82.8 mm
- net ROW2_MID: track 68.2 -> 70.0 mm
- net ROW1_MID: track 52.4 -> 53.3 mm
Other:
- board text added: "BACK"
- board text added: "C13 C12 C11 C10 C09 C08 C07 C06 C05 C04 C03 C02 C01 C00"
- board text added: "C16 C15 C14"
- board text added: "C20 C19 C18 C17"
- board text added: "FRONT"
- board text added: "R0"
- board text added: "R1 R2 R3 R4 R5"
- board text added: "umu!"
- board text added: "universa universis rev. 1 03-2023"

Commit message: start rounding corners
Parts:
- moved D90 9.68 mm to (467.0, 46.2), turned to 0 degrees
Routing:
- net Net-(D81-K): track 54.2 -> 44.5 mm
- net Net-(D90-A): track 17.5 -> 24.0 mm
Other:
- outline, holes or cut-outs redrawn

Commit message: finish rounding out corners.
Parts:
- moved D111 11.7 mm to (546.6, 142.8), turned to 0 degrees
- moved D93 9.81 mm to (466.9, 146.4), turned to 0 degrees
- moved D65 1.10 mm to (413.4, 146.5)
Routing:
- net ROW5_MID: track 129.6 -> 119.8 mm
- net ROW4_RIGHT: track 139.2 -> 130.9 mm
- net Net-(D93-A): track 7.84 -> 14.2 mm
- net COL14_BOTTOM: track 109.8 -> 115.5 mm
- net COL15_BOTTOM: track 90.8 -> 95.2 mm
- net Net-(D111-A): track 9.24 -> 11.7 mm
- net ROW5_LEFT: track 346.5 -> 345.0 mm
- net Net-(D65-A): track 12.5 -> 11.4 mm
Other:
- outline, holes or cut-outs redrawn
- board text added: "universa universis rev. 0/α 03-2023"
- board text removed: "universa universis rev. 1 03-2023"
